File: corne-ultralight/pcb/corne-ultralight.kicad_pcb (KiCad board)
At the start: 2 copper layers, 275.5 x 105.6 mm, 132 parts, among them J2 OLED, J5 Breakaway_Tabs, J7 OLED, SW1 SW_PUSH, SW10 SW_PUSH, SW11 SW_PUSH, SW12 SW_PUSH, SW13 SW_PUSH, SW14 SW_PUSH, SW15 SW_PUSH, SW16 SW_PUSH, SW17 SW_PUSH, SW18 SW_PUSH, SW19 SW_PUSH, SW2 SW_PUSH, SW20 SW_PUSH, SW21 SW_PUSH, SW22 SW_PUSH, SW23 SW_PUSH, SW24 SW_PUSH, SW25 SW_PUSH, SW26 SW_PUSH, SW27 SW_PUSH, SW28 SW_PUSH, SW29 SW_PUSH, SW3 SW_PUSH, SW30 SW_PUSH, SW31 SW_PUSH, SW32 SW_PUSH, SW33 SW_PUSH, SW34 SW_PUSH, SW35 SW_PUSH, SW36 SW_PUSH, SW37 SW_PUSH, SW38 SW_PUSH, SW39 SW_PUSH, SW4 SW_PUSH, SW40 SW_PUSH, SW41 SW_PUSH, SW42 SW_PUSH, SW5 SW_PUSH, SW6 SW_PUSH, SW7 SW_PUSH, SW8 SW_PUSH, SW9 SW_PUSH, U1 ProMicro, U2 ProMicro

Commit message: Mods to Ultra Light crkbd
Parts:
- removed BATJ1, BATJ3: Conn_01x02_Female, Connector_PinHeader_2.54mm:PinHeader_1x02_P2.54mm_Vertical
- removed the Ref** at (50.7, 74.4)
- removed the Ref** at (50.7, 55.4)
- removed the Ref** at (250.2, 74.4)
- removed the Ref** at (250.2, 55.4)
- SW1, SW10, SW11, SW12, SW13, SW14, SW15, SW16, SW17, SW18, SW19, SW2, SW20, SW22, SW23, SW24, SW25, SW26, SW27, SW28, SW29, SW3, SW30, SW31, SW32, SW33, SW34, SW35, SW36, SW37, SW38, SW39, SW4, SW40, SW41, SW5, SW6, SW7, SW8, SW9: footprint gateron-ks27:gateron-ks27-choc-v1-mx -> ScottoKeebs_Hotswap:Hotswap_Choc_V1V2_1.00u
- SW21, SW42: footprint gateron-ks27:gateron-ks27-choc-v1-mx-1.5u -> ScottoKeebs_Hotswap:Hotswap_Choc_V1V2_1.50u
- moved D21 26.3 mm to (123.2, 110.7), turned to 150 degrees
- moved D42 25.1 mm to (179.9, 112.2), turned to -150 degrees
- moved D20 22.5 mm to (117.8, 106.5), turned to 80 degrees
- moved D16 18.7 mm to (89.9, 79.2)
- moved D24 17.8 mm to (249.1, 47.7)
- moved D36 17.7 mm to (249.5, 84.7)
- moved D38 17.2 mm to (211.2, 83.6)
- moved D19 16.9 mm to (97.3, 100.7)
- moved D2 16.7 mm to (49.8, 47.9)
- moved D26 16.7 mm to (211.3, 43.2)
- moved D14 16.7 mm to (49.7, 85.9)
- moved D1 10.0 mm to (24.7, 54.3), turned to 0 degrees
- moved D40 9.40 mm to (218.6, 89.7), turned to 180 degrees
- moved D18 7.14 mm to (108.6, 86.0)
- moved D33 6.68 mm to (189.4, 66.2), turned to 0 degrees
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Connections:
- SW1 pad 2: Net-(D1-Pad2) -> Net-(D1-A)
- SW10 pad 2: Net-(D10-Pad2) -> Net-(D10-A)
- SW12 pad 2: Net-(D12-Pad2) -> Net-(D12-A)
- SW13 pad 2: Net-(D13-Pad2) -> Net-(D13-A)
- SW14 pad 2: Net-(D14-Pad2) -> Net-(D14-A)
- SW15 pad 2: Net-(D15-Pad2) -> Net-(D15-A)
- SW16 pad 2: Net-(D16-Pad2) -> Net-(D16-A)
- SW17 pad 2: Net-(D17-Pad2) -> Net-(D17-A)
- SW18 pad 2: Net-(D18-Pad2) -> Net-(D18-A)
- SW2 pad 2: Net-(D2-Pad2) -> Net-(D2-A)
- SW22 pad 2: Net-(D22-Pad2) -> Net-(D22-A)
- SW23 pad 2: Net-(D23-Pad2) -> Net-(D23-A)
- SW24 pad 2: Net-(D24-Pad2) -> Net-(D24-A)
- SW25 pad 2: Net-(D25-Pad2) -> Net-(D25-A)
- SW26 pad 2: Net-(D26-Pad2) -> Net-(D26-A)
- SW27 pad 2: Net-(D27-Pad2) -> Net-(D27-A)
- SW28 pad 2: Net-(D28-Pad2) -> Net-(D28-A)
- SW29 pad 2: Net-(D29-Pad2) -> Net-(D29-A)
- SW30 pad 2: Net-(D30-Pad2) -> Net-(D30-A)
- SW31 pad 2: Net-(D31-Pad2) -> Net-(D31-A)
- SW32 pad 2: Net-(D32-Pad2) -> Net-(D32-A)
- SW33 pad 2: Net-(D33-Pad2) -> Net-(D33-A)
- SW34 pad 2: Net-(D34-Pad2) -> Net-(D34-A)
- SW35 pad 2: Net-(D35-Pad2) -> Net-(D35-A)
- SW36 pad 2: Net-(D36-Pad2) -> Net-(D36-A)
- SW37 pad 2: Net-(D37-Pad2) -> Net-(D37-A)
- SW38 pad 2: Net-(D38-Pad2) -> Net-(D38-A)
- SW39 pad 2: Net-(D39-Pad2) -> Net-(D39-A)
- SW40 pad 2: Net-(D40-Pad2) -> Net-(D40-A)
- SW41 pad 2: Net-(D41-Pad2) -> Net-(D41-A)
- SW42 pad 2: Net-(D42-Pad2) -> Net-(D42-A)
- SW6 pad 2: Net-(D6-Pad2) -> Net-(D6-A)
- SW7 pad 2: Net-(D7-Pad2) -> Net-(D7-A)
- SW8 pad 2: Net-(D8-Pad2) -> Net-(D8-A)
- SW9 pad 2: Net-(D9-Pad2) -> Net-(D9-A)
Routing:
- net Net-(D42-Pad2): track 41.1 -> 0.00 mm
- net row3_r: track 88.1 -> 122.9 mm
- net col1: track 147.7 -> 177.9 mm, vias 1 -> 3
- net Net-(D1-A): track 0.00 -> 29.2 mm
- net Net-(BATJ1-Pin_2): track 33.1 -> 5.44 mm, vias 1 -> 0
- net GND: track 88.8 -> 62.1 mm
- net Net-(D22-A): track 0.00 -> 25.3 mm
- net Net-(D12-A): track 0.00 -> 23.7 mm, vias 0 -> 2
- net Net-(D35-Pad2): track 23.1 -> 0.00 mm, vias 1 -> 0
- net Net-(D29-Pad2): track 23.0 -> 0.00 mm, vias 1 -> 0
- net Net-(D10-A): track 0.00 -> 22.6 mm
- net row1: track 168.5 -> 146.1 mm
- net Net-(D28-A): track 0.00 -> 22.4 mm, vias 0 -> 2
- net Net-(D30-A): track 0.00 -> 22.0 mm
- net row1_r: track 139.8 -> 118.1 mm
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Other:
- board size 275.5 x 105.6 mm -> 276.5 x 105.6 mm
- board text added: "Corne UltraLight v2.0 PCB, modded by alopo."
- board text added: "J5"
- board text removed: "Corne Light v2.0 PCB Designed by foostan"
- board text removed: "Corne UltraLight v2.0 PCB Designed by foostan, mods by petejohanson"
